File: electrical/kicad/4_indicator_driver/4_indicator_driver.kicad_sch (KiCad schematic)
At the start: 33 parts, among them J1 Conn_01x04, J2 Conn_01x02, J3 Conn_01x02, J4 Conn_01x03, Q1 IRLZ44N, Q10 BC817, Q2 IRLZ44N, Q3 IRLZ44N, Q4 IRLZ44N, Q5 IRLZ44N, Q6 BC817, Q7 BC817, Q8 BC817, Q9 BC817

Commit message: final electric schematics
Parts:
- removed C1: 100nF, symbol Device:C
- removed D1: D, Package_SON:WSON-8-1EP_6x5mm_P1.27mm_EP3.4x4mm, symbol Device:D
- removed J4: Conn_01x03, Package_TO_SOT_SMD:TO-263-9_TabPin5, symbol Connector_Generic:Conn_01x03
- removed R16: 1K, symbol Device:R
